Commit message: all joint of robot spawn successfully on gazebo

File: urdf/robot.urdf (robot description, URDF)
Before this commit: robot robot, 4 links, 3 joints
Joints:
- added joint slider_joint: type prismatic, parent base_link, child hip_link, origin xyz=0 0 0 rpy=0 0 0, axis 0 0 0.5, limit lower=0 upper=1 effort=1000 velocity=100

File: urdf/robot_for_sim.urdf (robot description, URDF)
Before this commit: robot robot, 5 links, 4 joints
Joints:
- removed joint world_to_base
- added joint base_to_hip: type fixed, parent base_link, child hip_link, origin xyz=0 0 0 rpy=0 0 0
- joint slider_joint: child hip_link -> base_link; limit lower=0 upper=1 effort=1000 velocity=100 -> lower=0 upper=5 effort=1000 velocity=100; parent base_link -> world
