Commit message: fix effort limit

File: urdf/robot_for_sim.urdf (robot description, URDF)
Before this commit: robot robot, 5 links, 4 joints
Joints:
- joint hip_to_thigh: limit lower=-1.04719732679 upper=0.523599 effort=1000 velocity=10 -> lower=-1.04719732679 upper=0.523599 effort=10000 velocity=10
- joint slider_joint: limit lower=0 upper=5 effort=1000 velocity=100 -> lower=0 upper=5 effort=10000 velocity=100
- joint thigh_to_shin: limit lower=-0.523599 upper=2.61799732679 effort=1000 velocity=10 -> lower=-0.523599 upper=2.61799732679 effort=10000 velocity=10
